File: pcb/Power_control.kicad_sch (KiCad schematic)
At the start: 3 parts, among them U13 MIC94300

Commit message: Schema & PCB: reconect output of charger from SNS to VBAT
Other:
- company: (none) -> Author: Petr Malaník
- title: (none) -> Kratos pack
Changed lines of the file:
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@@
 (kicad_sch (version 20211123) (generator eeschema)
   (paper "A4")
+  (title_block
+    (title "Kratos pack")
+    (date "2022-07-01")
+    (rev "v1.1")
+    (company "Author: Petr Malaník")
+  )
   (junction (at 128.27 96.52) (diameter 1.016) (color 0 0 0 0)
   )

Commit message: PCB: change footprint of resistors and capacitors to smaller version
After first version is apparent that smaller footprint used on some
resistors are big enough for manual soldering. Because of this was
exchanged for custom smaller version.

In current version pull-up resistor of reset circuit is not connected,
because is mend to be removed in future.
Parts:
- C29, C30: footprint Capacitor_SMD:C_0603_1608Metric -> TCY_passives:C_0603_1608Metric
Changed lines of the file:
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@@
       (effects (font (size 1.27 1.27)) (justify left))
     )
-    (property "Footprint" "Capacitor_SMD:C_0603_1608Metric" (id 2) (at 110.1852 97.79 0)
+    (property "Footprint" "TCY_passives:C_0603_1608Metric" (id 2) (at 110.1852 97.79 0)
       (effects (font (size 1.27 1.27)) hide)
     )
@@
       (effects (font (size 1.27 1.27)) (justify left))
     )
-    (property "Footprint" "Capacitor_SMD:C_0603_1608Metric" (id 2) (at 141.9352 97.79 0)
+    (property "Footprint" "TCY_passives:C_0603_1608Metric" (id 2) (at 141.9352 97.79 0)
       (effects (font (size 1.27 1.27)) hide)
     )
