File: pcb/Power_control.kicad_sch (KiCad schematic)
At the start: 3 parts, among them U13 MIC94300

Commit message: Schema & PCB: Fix USB detection by MCU and USB converter, hide GND labels
USB detection circuit is now connected only to MCU.
Converter from USB to UART (CP2102) is directly connected to VBUS.
Changed lines of the file:
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@@
       (effects (font (size 1.27 1.27)) hide)
     )
-    (property "Value" "GND" (id 1) (at 128.3843 102.1144 0))
+    (property "Value" "GND" (id 1) (at 128.3843 102.1144 0)
+      (effects (font (size 1.27 1.27)) hide)
+    )
     (property "Footprint" "" (id 2) (at 128.27 97.79 0)
       (effects (font (size 1.27 1.27)) hide)
@@
       (effects (font (size 1.27 1.27)) hide)
     )
-    (property "Value" "GND" (id 1) (at 109.3343 102.1144 0))
+    (property "Value" "GND" (id 1) (at 109.3343 102.1144 0)
+      (effects (font (size 1.27 1.27)) hide)
+    )
     (property "Footprint" "" (id 2) (at 109.22 97.79 0)
       (effects (font (size 1.27 1.27)) hide)
@@
       (effects (font (size 1.27 1.27)) hide)
     )
-    (property "Value" "GND" (id 1) (at 141.0843 102.1144 0))
+    (property "Value" "GND" (id 1) (at 141.0843 102.1144 0)
+      (effects (font (size 1.27 1.27)) hide)
+    )
     (property "Footprint" "" (id 2) (at 140.97 97.79 0)
       (effects (font (size 1.27 1.27)) hide)
