File: pcb/BTN_Denoise.kicad_sch (KiCad schematic)
At the start: 5 parts, among them U12 74LVC2G14

Commit message: Schema: Remove unnecessary test points (switches) and filtering capacitors (STM, CP2102)
Parts:
- removed TP11: TestPoint, TestPoint:TestPoint_Pad_D1.0mm, symbol Connector:TestPoint
- TP12: footprint TestPoint:TestPoint_Pad_D1.0mm -> TCY_connectors:TestPoint_Pad_D0.5mm
- U12: footprint (none) -> Package_TO_SOT_SMD:SOT-363_SC-70-6
Changed lines of the file:
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@@
     (effects (font (size 1.27 1.27)) (justify left))
-  )
-  (symbol (lib_id "Connector:TestPoint") (at 117.475 87.63 0)
-    (in_bom yes) (on_board yes)
-    (property "Reference" "TP11" (id 0) (at 115.57 81.915 0)
-      (effects (font (size 1.27 1.27)) (justify left))
-    )
-    (property "Value" "TestPoint" (id 1) (at 119.38 86.995 0)
-      (effects (font (size 1.27 1.27)) (justify left) hide)
-    )
-    (property "Footprint" "TestPoint:TestPoint_Pad_D1.0mm" (id 2) (at 122.555 87.63 0)
-      (effects (font (size 1.27 1.27)) hide)
-    )
-    (property "Datasheet" "~" (id 3) (at 122.555 87.63 0)
-      (effects (font (size 1.27 1.27)) hide)
-    )
   )
   (symbol (lib_id "Connector:TestPoint") (at 137.16 87.63 0)
@@
       (effects (font (size 1.27 1.27)) (justify left) hide)
     )
-    (property "Footprint" "TestPoint:TestPoint_Pad_D1.0mm" (id 2) (at 142.24 87.63 0)
+    (property "Footprint" "TCY_connectors:TestPoint_Pad_D0.5mm" (id 2) (at 142.24 87.63 0)
       (effects (font (size 1.27 1.27)) hide)
     )
@@
     (property "Reference" "U12" (id 0) (at 135.255 89.516 0))
     (property "Value" "74LVC2G14" (id 1) (at 137.795 91.8145 0))
-    (property "Footprint" "" (id 2) (at 130.81 87.63 0)
+    (property "Footprint" "Package_TO_SOT_SMD:SOT-363_SC-70-6" (id 2) (at 130.81 87.63 0)
       (effects (font (size 1.27 1.27)) hide)
     )

Commit message: Schema: add some connection STM32, remove redundant connections to BQ25887
Parts:
- renumbered C27 to C28, R35 to R36, TP12 to TP14
Changed lines of the file:
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@@
   (symbol (lib_id "Connector:TestPoint") (at 137.16 87.63 0)
     (in_bom yes) (on_board yes)
-    (property "Reference" "TP12" (id 0) (at 139.065 83.185 0)
+    (property "Reference" "TP14" (id 0) (at 139.065 83.185 0)
       (effects (font (size 1.27 1.27)) (justify left))
     )
@@
   (symbol (lib_id "power:+3V3") (at 130.81 83.82 0)
     (in_bom yes) (on_board yes)
-    (property "Reference" "#PWR085" (id 0) (at 130.81 87.63 0)
+    (property "Reference" "#PWR088" (id 0) (at 130.81 87.63 0)
       (effects (font (size 1.27 1.27)) hide)
     )
@@
   (symbol (lib_id "power:GND") (at 117.475 95.25 0)
     (in_bom yes) (on_board yes)
-    (property "Reference" "#PWR083" (id 0) (at 117.475 101.6 0)
+    (property "Reference" "#PWR086" (id 0) (at 117.475 101.6 0)
       (effects (font (size 1.27 1.27)) hide)
     )
@@
   (symbol (lib_id "power:GND") (at 130.81 91.44 0)
     (in_bom yes) (on_board yes)
-    (property "Reference" "#PWR084" (id 0) (at 130.81 97.79 0)
+    (property "Reference" "#PWR087" (id 0) (at 130.81 97.79 0)
       (effects (font (size 1.27 1.27)) hide)
     )
@@
   (symbol (lib_id "Device:R") (at 111.76 87.63 270)
     (in_bom yes) (on_board yes)
-    (property "Reference" "R35" (id 0) (at 111.76 82.3722 90))
+    (property "Reference" "R36" (id 0) (at 111.76 82.3722 90))
     (property "Value" "1k" (id 1) (at 111.76 84.6836 90))
     (property "Footprint" "Resistor_SMD:R_0603_1608Metric" (id 2) (at 111.76 85.852 90)
@@
   (symbol (lib_id "Device:C") (at 117.475 91.44 0)
     (in_bom yes) (on_board yes)
-    (property "Reference" "C27" (id 0) (at 120.396 90.2716 0)
+    (property "Reference" "C28" (id 0) (at 120.396 90.2716 0)
       (effects (font (size 1.27 1.27)) (justify left))
     )

Commit message: Schema: update connection of CS_EN pin
Parts:
- renumbered C28 to C27, R36 to R35, TP14 to TP12
Changed lines of the file:
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@@
   (symbol (lib_id "Connector:TestPoint") (at 137.16 87.63 0)
     (in_bom yes) (on_board yes)
-    (property "Reference" "TP14" (id 0) (at 139.065 83.185 0)
+    (property "Reference" "TP12" (id 0) (at 139.065 83.185 0)
       (effects (font (size 1.27 1.27)) (justify left))
     )
@@
   (symbol (lib_id "Device:R") (at 111.76 87.63 270)
     (in_bom yes) (on_board yes)
-    (property "Reference" "R36" (id 0) (at 111.76 82.3722 90))
+    (property "Reference" "R35" (id 0) (at 111.76 82.3722 90))
     (property "Value" "1k" (id 1) (at 111.76 84.6836 90))
     (property "Footprint" "Resistor_SMD:R_0603_1608Metric" (id 2) (at 111.76 85.852 90)
@@
   (symbol (lib_id "Device:C") (at 117.475 91.44 0)
     (in_bom yes) (on_board yes)
-    (property "Reference" "C28" (id 0) (at 120.396 90.2716 0)
+    (property "Reference" "C27" (id 0) (at 120.396 90.2716 0)
       (effects (font (size 1.27 1.27)) (justify left))
     )

Commit message: PCB: add 3D packages to parts
Parts:
- renumbered C27 to C28, R35 to R36, TP12 to TP14
Changed lines of the file:
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@@
   (symbol (lib_id "Connector:TestPoint") (at 137.16 87.63 0)
     (in_bom yes) (on_board yes)
-    (property "Reference" "TP12" (id 0) (at 139.065 83.185 0)
+    (property "Reference" "TP14" (id 0) (at 139.065 83.185 0)
       (effects (font (size 1.27 1.27)) (justify left))
     )
@@
   (symbol (lib_id "Device:R") (at 111.76 87.63 270)
     (in_bom yes) (on_board yes)
-    (property "Reference" "R35" (id 0) (at 111.76 82.3722 90))
+    (property "Reference" "R36" (id 0) (at 111.76 82.3722 90))
     (property "Value" "1k" (id 1) (at 111.76 84.6836 90))
     (property "Footprint" "Resistor_SMD:R_0603_1608Metric" (id 2) (at 111.76 85.852 90)
@@
   (symbol (lib_id "Device:C") (at 117.475 91.44 0)
     (in_bom yes) (on_board yes)
-    (property "Reference" "C27" (id 0) (at 120.396 90.2716 0)
+    (property "Reference" "C28" (id 0) (at 120.396 90.2716 0)
       (effects (font (size 1.27 1.27)) (justify left))
     )

Commit message: Schema & PCB: add pull up to wakeup button
Parts:
- added R43: R, TCY_passives:R_0603_1608Metric, symbol Device:R
- renumbered C28 to C27, R36 to R35, TP14 to TP12
Connections:
- net +3V3: now also R43.1
- net IN: now also R43.2
Changed lines of the file:
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@@
 (kicad_sch (version 20201015) (generator eeschema)
   (paper "A4")
+  (junction (at 106.68 87.63) (diameter 1.016) (color 0 0 0 0))
   (junction (at 117.475 87.63) (diameter 1.016) (color 0 0 0 0))
   (junction (at 137.16 87.63) (diameter 1.016) (color 0 0 0 0))
-  (wire (pts (xy 105.41 87.63) (xy 107.95 87.63))
+  (wire (pts (xy 105.41 87.63) (xy 106.68 87.63))
+    (stroke (width 0) (type solid) (color 0 0 0 0))
+  )
+  (wire (pts (xy 106.68 85.09) (xy 106.68 87.63))
+    (stroke (width 0) (type solid) (color 0 0 0 0))
+  )
+  (wire (pts (xy 106.68 87.63) (xy 107.95 87.63))
     (stroke (width 0) (type solid) (color 0 0 0 0))
   )
@@
   (symbol (lib_id "Connector:TestPoint") (at 137.16 87.63 0)
     (in_bom yes) (on_board yes)
-    (property "Reference" "TP14" (id 0) (at 139.065 83.185 0)
+    (property "Reference" "TP12" (id 0) (at 139.065 83.185 0)
       (effects (font (size 1.27 1.27)) (justify left))
     )
@@
     )
   )
+  (symbol (lib_id "power:+3V3") (at 106.68 77.47 0)
+    (in_bom yes) (on_board yes)
+    (property "Reference" "#PWR0109" (id 0) (at 106.68 81.28 0)
+      (effects (font (size 1.27 1.27)) hide)
+    )
+    (property "Value" "+3V3" (id 1) (at 107.0483 73.1456 0))
+    (property "Footprint" "" (id 2) (at 106.68 77.47 0)
+      (effects (font (size 1.27 1.27)) hide)
+    )
+    (property "Datasheet" "" (id 3) (at 106.68 77.47 0)
+      (effects (font (size 1.27 1.27)) hide)
+    )
+  )
   (symbol (lib_id "power:+3V3") (at 130.81 83.82 0)
     (in_bom yes) (on_board yes)
-    (property "Reference" "#PWR088" (id 0) (at 130.81 87.63 0)
+    (property "Reference" "#PWR085" (id 0) (at 130.81 87.63 0)
       (effects (font (size 1.27 1.27)) hide)
     )
@@
   (symbol (lib_id "power:GND") (at 117.475 95.25 0)
     (in_bom yes) (on_board yes)
-    (property "Reference" "#PWR086" (id 0) (at 117.475 101.6 0)
+    (property "Reference" "#PWR083" (id 0) (at 117.475 101.6 0)
       (effects (font (size 1.27 1.27)) hide)
     )
@@
   (symbol (lib_id "power:GND") (at 130.81 91.44 0)
     (in_bom yes) (on_board yes)
-    (property "Reference" "#PWR087" (id 0) (at 130.81 97.79 0)
+    (property "Reference" "#PWR084" (id 0) (at 130.81 97.79 0)
       (effects (font (size 1.27 1.27)) hide)
     )
@@
     )
   )
+  (symbol (lib_id "Device:R") (at 106.68 81.28 0)
+    (in_bom yes) (on_board yes)
+    (property "Reference" "R43" (id 0) (at 108.4581 80.1306 0)
+      (effects (font (size 1.27 1.27)) (justify left))
+    )
+    (property "Value" "R" (id 1) (at 108.4581 82.4293 0)
+      (effects (font (size 1.27 1.27)) (justify left))
+    )
+    (property "Footprint" "TCY_passives:R_0603_1608Metric" (id 2) (at 104.902 81.28 90)
+      (effects (font (size 1.27 1.27)) hide)
+    )
+    (property "Datasheet" "~" (id 3) (at 106.68 81.28 0)
+      (effects (font (size 1.27 1.27)) hide)
+    )
+  )
   (symbol (lib_id "Device:R") (at 111.76 87.63 270)
     (in_bom yes) (on_board yes)
-    (property "Reference" "R36" (id 0) (at 111.76 82.3722 90))
-    (property "Value" "1k" (id 1) (at 111.76 84.6836 90))
+    (property "Reference" "R35" (id 0) (at 109.22 89.9922 90))
+    (property "Value" "1k" (id 1) (at 113.03 89.7636 90))
     (property "Footprint" "Resistor_SMD:R_0603_1608Metric" (id 2) (at 111.76 85.852 90)
       (effects (font (size 1.27 1.27)) hide)
@@
   (symbol (lib_id "Device:C") (at 117.475 91.44 0)
     (in_bom yes) (on_board yes)
-    (property "Reference" "C28" (id 0) (at 120.396 90.2716 0)
+    (property "Reference" "C27" (id 0) (at 120.396 90.2716 0)
       (effects (font (size 1.27 1.27)) (justify left))
     )

Commit message: Schema: update page layout and add I2C addresses to I2C device
Parts:
- R43: value R -> 470k
Changed lines of the file:
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@@
-(kicad_sch (version 20201015) (generator eeschema)
+(kicad_sch (version 20211123) (generator eeschema)
   (paper "A4")
-  (junction (at 106.68 87.63) (diameter 1.016) (color 0 0 0 0))
-  (junction (at 117.475 87.63) (diameter 1.016) (color 0 0 0 0))
-  (junction (at 137.16 87.63) (diameter 1.016) (color 0 0 0 0))
-  (wire (pts (xy 105.41 87.63) (xy 106.68 87.63))
+  (junction (at 137.16 87.63) (diameter 1.016) (color 0 0 0 0)
+  )
+  (junction (at 106.68 87.63) (diameter 1.016) (color 0 0 0 0)
+  )
+  (junction (at 117.475 87.63) (diameter 1.016) (color 0 0 0 0)
+  )
+  (wire (pts (xy 106.68 87.63) (xy 107.95 87.63))
+    (stroke (width 0) (type solid) (color 0 0 0 0))
+  )
+  (wire (pts (xy 142.24 87.63) (xy 137.16 87.63))
+    (stroke (width 0) (type solid) (color 0 0 0 0))
+  )
+  (wire (pts (xy 115.57 87.63) (xy 117.475 87.63))
     (stroke (width 0) (type solid) (color 0 0 0 0))
   )
@@
     (stroke (width 0) (type solid) (color 0 0 0 0))
   )
-  (wire (pts (xy 106.68 87.63) (xy 107.95 87.63))
-    (stroke (width 0) (type solid) (color 0 0 0 0))
-  )
-  (wire (pts (xy 115.57 87.63) (xy 117.475 87.63))
+  (wire (pts (xy 105.41 87.63) (xy 106.68 87.63))
     (stroke (width 0) (type solid) (color 0 0 0 0))
   )
   (wire (pts (xy 117.475 87.63) (xy 123.19 87.63))
-    (stroke (width 0) (type solid) (color 0 0 0 0))
-  )
-  (wire (pts (xy 142.24 87.63) (xy 137.16 87.63))
     (stroke (width 0) (type solid) (color 0 0 0 0))
   )
@@
     (effects (font (size 1.27 1.27)) (justify left))
   )
-  (symbol (lib_id "Connector:TestPoint") (at 137.16 87.63 0)
+  (symbol (lib_id "power:GND") (at 117.475 95.25 0) (unit 1)
+    (in_bom yes) (on_board yes)
+    (property "Reference" "#PWR083" (id 0) (at 117.475 101.6 0)
+      (effects (font (size 1.27 1.27)) hide)
+    )
+    (property "Value" "GND" (id 1) (at 117.475 99.06 0))
+    (property "Footprint" "" (id 2) (at 117.475 95.25 0)
+      (effects (font (size 1.27 1.27)) hide)
+    )
+    (property "Datasheet" "" (id 3) (at 117.475 95.25 0)
+      (effects (font (size 1.27 1.27)) hide)
+    )
+    (pin "1")
+  )
+  (symbol (lib_id "74xGxx:74LVC2G14") (at 130.81 87.63 0) (unit 1)
+    (in_bom yes) (on_board yes)
+    (property "Reference" "U12" (id 0) (at 135.255 89.516 0))
+    (property "Value" "74LVC2G14" (id 1) (at 137.795 91.8145 0))
+    (property "Footprint" "Package_TO_SOT_SMD:SOT-363_SC-70-6" (id 2) (at 130.81 87.63 0)
+      (effects (font (size 1.27 1.27)) hide)
+    )
+    (property "Datasheet" "https://www.ti.com/lit/ds/symlink/sn74lvc2g14.pdf" (id 3) (at 130.81 87.63 0)
+      (effects (font (size 1.27 1.27)) hide)
+    )
+    (pin "2")
+    (pin "5")
+    (pin "1")
+    (pin "6")
+    (pin "3")
+    (pin "4")
+  )
+  (symbol (lib_id "Device:C") (at 117.475 91.44 0) (unit 1)
+    (in_bom yes) (on_board yes)
+    (property "Reference" "C27" (id 0) (at 120.396 90.2716 0)
+      (effects (font (size 1.27 1.27)) (justify left))
+    )
+    (property "Value" "100nF" (id 1) (at 120.396 92.583 0)
+      (effects (font (size 1.27 1.27)) (justify left))
+    )
+    (property "Footprint" "Capacitor_SMD:C_0603_1608Metric" (id 2) (at 118.4402 95.25 0)
+      (effects (font (size 1.27 1.27)) hide)
+    )
+    (property "Datasheet" "~" (id 3) (at 117.475 91.44 0)
+      (effects (font (size 1.27 1.27)) hide)
+    )
+    (pin "1")
+    (pin "2")
+  )
+  (symbol (lib_id "power:+3V3") (at 106.68 77.47 0) (unit 1)
+    (in_bom yes) (on_board yes)
+    (property "Reference" "#PWR0109" (id 0) (at 106.68 81.28 0)
+      (effects (font (size 1.27 1.27)) hide)
+    )
+    (property "Value" "+3V3" (id 1) (at 107.0483 73.1456 0))
+    (property "Footprint" "" (id 2) (at 106.68 77.47 0)
+      (effects (font (size 1.27 1.27)) hide)
+    )
+    (property "Datasheet" "" (id 3) (at 106.68 77.47 0)
+      (effects (font (size 1.27 1.27)) hide)
+    )
+    (pin "1")
+  )
+  (symbol (lib_id "Device:R") (at 111.76 87.63 270) (unit 1)
+    (in_bom yes) (on_board yes)
+    (property "Reference" "R35" (id 0) (at 109.22 89.9922 90))
+    (property "Value" "1k" (id 1) (at 113.03 89.7636 90))
+    (property "Footprint" "Resistor_SMD:R_0603_1608Metric" (id 2) (at 111.76 85.852 90)
+      (effects (font (size 1.27 1.27)) hide)
+    )
+    (property "Datasheet" "~" (id 3) (at 111.76 87.63 0)
+      (effects (font (size 1.27 1.27)) hide)
+    )
+    (pin "1")
+    (pin "2")
+  )
+  (symbol (lib_id "Connector:TestPoint") (at 137.16 87.63 0) (unit 1)
     (in_bom yes) (on_board yes)
     (property "Reference" "TP12" (id 0) (at 139.065 83.185 0)
@@
       (effects (font (size 1.27 1.27)) hide)
     )
+    (pin "1")
   )
-  (symbol (lib_id "power:+3V3") (at 106.68 77.47 0)
+  (symbol (lib_id "Device:R") (at 106.68 81.28 0) (unit 1)
     (in_bom yes) (on_board yes)
-    (property "Reference" "#PWR0110" (id 0) (at 106.68 81.28 0)
+    (property "Reference" "R43" (id 0) (at 108.4581 80.1306 0)
+      (effects (font (size 1.27 1.27)) (justify left))
+    )
+    (property "Value" "470k" (id 1) (at 108.4581 82.4293 0)
+      (effects (font (size 1.27 1.27)) (justify left))
+    )
+    (property "Footprint" "TCY_passives:R_0603_1608Metric" (id 2) (at 104.902 81.28 90)
       (effects (font (size 1.27 1.27)) hide)
     )
-    (property "Value" "+3V3" (id 1) (at 107.0483 73.1456 0))
-    (property "Footprint" "" (id 2) (at 106.68 77.47 0)
+    (property "Datasheet" "~" (id 3) (at 106.68 81.28 0)
       (effects (font (size 1.27 1.27)) hide)
     )
-    (property "Datasheet" "" (id 3) (at 106.68 77.47 0)
-      (effects (font (size 1.27 1.27)) hide)
-    )
+    (pin "1")
+    (pin "2")
   )
-  (symbol (lib_id "power:+3V3") (at 130.81 83.82 0)
+  (symbol (lib_id "power:+3V3") (at 130.81 83.82 0) (unit 1)
     (in_bom yes) (on_board yes)
-    (property "Reference" "#PWR088" (id 0) (at 130.81 87.63 0)
+    (property "Reference" "#PWR085" (id 0) (at 130.81 87.63 0)
       (effects (font (size 1.27 1.27)) hide)
     )
@@
       (effects (font (size 1.27 1.27)) hide)
     )
+    (pin "1")
   )
-  (symbol (lib_id "power:GND") (at 117.475 95.25 0)
+  (symbol (lib_id "power:GND") (at 130.81 91.44 0) (unit 1)
     (in_bom yes) (on_board yes)
-    (property "Reference" "#PWR086" (id 0) (at 117.475 101.6 0)
-      (effects (font (size 1.27 1.27)) hide)
-    )
-    (property "Value" "GND" (id 1) (at 117.475 99.06 0))
-    (property "Footprint" "" (id 2) (at 117.475 95.25 0)
-      (effects (font (size 1.27 1.27)) hide)
-    )
-    (property "Datasheet" "" (id 3) (at 117.475 95.25 0)
-      (effects (font (size 1.27 1.27)) hide)
-    )
-  )
-  (symbol (lib_id "power:GND") (at 130.81 91.44 0)
-    (in_bom yes) (on_board yes)
-    (property "Reference" "#PWR087" (id 0) (at 130.81 97.79 0)
+    (property "Reference" "#PWR084" (id 0) (at 130.81 97.79 0)
       (effects (font (size 1.27 1.27)) hide)
     )
@@
       (effects (font (size 1.27 1.27)) hide)
     )
-  )
-  (symbol (lib_id "Device:R") (at 106.68 81.28 0)
-    (in_bom yes) (on_board yes)
-    (property "Reference" "R43" (id 0) (at 108.4581 80.1306 0)
-      (effects (font (size 1.27 1.27)) (justify left))
-    )
-    (property "Value" "R" (id 1) (at 108.4581 82.4293 0)
-      (effects (font (size 1.27 1.27)) (justify left))
-    )
-    (property "Footprint" "TCY_passives:R_0603_1608Metric" (id 2) (at 104.902 81.28 90)
-      (effects (font (size 1.27 1.27)) hide)
-    )
-    (property "Datasheet" "~" (id 3) (at 106.68 81.28 0)
-      (effects (font (size 1.27 1.27)) hide)
-    )
-  )
-  (symbol (lib_id "Device:R") (at 111.76 87.63 270)
-    (in_bom yes) (on_board yes)
-    (property "Reference" "R35" (id 0) (at 109.22 89.9922 90))
-    (property "Value" "1k" (id 1) (at 113.03 89.7636 90))
-    (property "Footprint" "Resistor_SMD:R_0603_1608Metric" (id 2) (at 111.76 85.852 90)
-      (effects (font (size 1.27 1.27)) hide)
-    )
-    (property "Datasheet" "~" (id 3) (at 111.76 87.63 0)
-      (effects (font (size 1.27 1.27)) hide)
-    )
-  )
-  (symbol (lib_id "Device:C") (at 117.475 91.44 0)
-    (in_bom yes) (on_board yes)
-    (property "Reference" "C27" (id 0) (at 120.396 90.2716 0)
-      (effects (font (size 1.27 1.27)) (justify left))
-    )
-    (property "Value" "100nF" (id 1) (at 120.396 92.583 0)
-      (effects (font (size 1.27 1.27)) (justify left))
-    )
-    (property "Footprint" "Capacitor_SMD:C_0603_1608Metric" (id 2) (at 118.4402 95.25 0)
-      (effects (font (size 1.27 1.27)) hide)
-    )
-    (property "Datasheet" "~" (id 3) (at 117.475 91.44 0)
-      (effects (font (size 1.27 1.27)) hide)
-    )
-  )
-  (symbol (lib_id "74xGxx:74LVC2G14") (at 130.81 87.63 0)
-    (in_bom yes) (on_board yes)
-    (property "Reference" "U12" (id 0) (at 135.255 89.516 0))
-    (property "Value" "74LVC2G14" (id 1) (at 137.795 91.8145 0))
-    (property "Footprint" "Package_TO_SOT_SMD:SOT-363_SC-70-6" (id 2) (at 130.81 87.63 0)
-      (effects (font (size 1.27 1.27)) hide)
-    )
-    (property "Datasheet" "https://www.ti.com/lit/ds/symlink/sn74lvc2g14.pdf" (id 3) (at 130.81 87.63 0)
-      (effects (font (size 1.27 1.27)) hide)
-    )
+    (pin "1")
   )
 )
