File: pcb/Voltage_measuring.kicad_sch (KiCad schematic)
At the start: 4 parts, among them Q4 UT6MA2TCR

Commit message: Schema: update footprint 3-pin connectors, project cleanup, add gitignore
Parts:
- renumbered Q4 to Q6, R33 to R39, R34 to R40
Changed lines of the file:
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@@
   (symbol (lib_id "Device:R") (at 93.98 107.95 0)
     (in_bom yes) (on_board yes)
-    (property "Reference" "R33" (id 0) (at 95.7581 106.8006 0)
+    (property "Reference" "R39" (id 0) (at 95.7581 106.8006 0)
       (effects (font (size 1.27 1.27)) (justify left))
     )
@@
   (symbol (lib_id "Device:R") (at 101.6 88.9 0)
     (in_bom yes) (on_board yes)
-    (property "Reference" "R34" (id 0) (at 103.3781 87.7506 0)
+    (property "Reference" "R40" (id 0) (at 103.3781 87.7506 0)
       (effects (font (size 1.27 1.27)) (justify left))
     )
@@
   (symbol (lib_id "TCY_IC:UT6MA2TCR") (at 99.06 100.33 0)
     (in_bom yes) (on_board yes)
-    (property "Reference" "Q4" (id 0) (at 95.3771 94.1006 0)
+    (property "Reference" "Q6" (id 0) (at 95.3771 94.1006 0)
       (effects (font (size 1.27 1.27)) (justify left))
     )
@@
   (symbol (lib_id "TCY_IC:UT6MA2TCR") (at 109.22 92.71 0)
     (in_bom yes) (on_board yes)
-    (property "Reference" "Q4" (id 0) (at 113.1571 85.2106 0)
+    (property "Reference" "Q6" (id 0) (at 113.1571 85.2106 0)
       (effects (font (size 1.27 1.27)) (justify left))
     )

Commit message: Schema: update page layout and add I2C addresses to I2C device
Parts:
- renumbered Q6 to Q4, R39 to R33, R40 to R34
Connections:
- net DIV: now also Q4.3 (DP); no longer Q4.1 (SN)
- net IN: now also Q4.4 (SP), Q4.8 (SP); no longer Q4.6 (DN), Q4.7 (DN)
- net at Q4.6 (DN), Q4.7 (DN), R34.2: now also Q4.5 (GP); no longer Q4.2 (GN)
Changed lines of the file:
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@@
-(kicad_sch (version 20201015) (generator eeschema)
+(kicad_sch (version 20211123) (generator eeschema)
   (paper "A4")
-  (junction (at 93.98 100.33) (diameter 1.016) (color 0 0 0 0))
-  (junction (at 101.6 85.09) (diameter 1.016) (color 0 0 0 0))
-  (junction (at 101.6 92.71) (diameter 1.016) (color 0 0 0 0))
-  (wire (pts (xy 88.9 85.09) (xy 101.6 85.09))
-    (stroke (width 0) (type solid) (color 0 0 0 0))
+  (junction (at 101.6 85.09) (diameter 1.016) (color 0 0 0 0)
+  )
+  (junction (at 101.6 92.71) (diameter 1.016) (color 0 0 0 0)
+  )
+  (junction (at 93.98 100.33) (diameter 1.016) (color 0 0 0 0)
   )
   (wire (pts (xy 88.9 100.33) (xy 93.98 100.33))
-    (stroke (width 0) (type solid) (color 0 0 0 0))
-  )
-  (wire (pts (xy 93.98 100.33) (xy 93.98 104.14))
-    (stroke (width 0) (type solid) (color 0 0 0 0))
-  )
-  (wire (pts (xy 93.98 111.76) (xy 93.98 115.57))
-    (stroke (width 0) (type solid) (color 0 0 0 0))
-  )
-  (wire (pts (xy 101.6 85.09) (xy 111.76 85.09))
-    (stroke (width 0) (type solid) (color 0 0 0 0))
-  )
-  (wire (pts (xy 101.6 92.71) (xy 101.6 95.25))
-    (stroke (width 0) (type solid) (color 0 0 0 0))
-  )
-  (wire (pts (xy 101.6 105.41) (xy 101.6 115.57))
-    (stroke (width 0) (type solid) (color 0 0 0 0))
-  )
-  (wire (pts (xy 104.14 92.71) (xy 101.6 92.71))
     (stroke (width 0) (type solid) (color 0 0 0 0))
   )
@@
     (stroke (width 0) (type solid) (color 0 0 0 0))
   )
+  (wire (pts (xy 93.98 111.76) (xy 93.98 115.57))
+    (stroke (width 0) (type solid) (color 0 0 0 0))
+  )
+  (wire (pts (xy 93.98 100.33) (xy 93.98 104.14))
+    (stroke (width 0) (type solid) (color 0 0 0 0))
+  )
+  (wire (pts (xy 104.14 92.71) (xy 101.6 92.71))
+    (stroke (width 0) (type solid) (color 0 0 0 0))
+  )
+  (wire (pts (xy 101.6 92.71) (xy 101.6 95.25))
+    (stroke (width 0) (type solid) (color 0 0 0 0))
+  )
+  (wire (pts (xy 101.6 105.41) (xy 101.6 115.57))
+    (stroke (width 0) (type solid) (color 0 0 0 0))
+  )
+  (wire (pts (xy 88.9 85.09) (xy 101.6 85.09))
+    (stroke (width 0) (type solid) (color 0 0 0 0))
+  )
+  (wire (pts (xy 101.6 85.09) (xy 111.76 85.09))
+    (stroke (width 0) (type solid) (color 0 0 0 0))
+  )
   (hierarchical_label "IN" (shape input) (at 88.9 85.09 180)
     (effects (font (size 1.27 1.27)) (justify right))
@@
     (effects (font (size 1.27 1.27)) (justify left))
   )
-  (symbol (lib_id "power:GND") (at 93.98 115.57 0)
+  (symbol (lib_id "power:GND") (at 93.98 115.57 0) (unit 1)
     (in_bom yes) (on_board yes)
-    (property "Reference" "#PWR091" (id 0) (at 93.98 121.92 0)
+    (property "Reference" "#PWR078" (id 0) (at 93.98 121.92 0)
       (effects (font (size 1.27 1.27)) hide)
     )
@@
       (effects (font (size 1.27 1.27)) hide)
     )
+    (pin "1")
   )
-  (symbol (lib_id "power:GND") (at 101.6 115.57 0)
+  (symbol (lib_id "power:GND") (at 101.6 115.57 0) (unit 1)
     (in_bom yes) (on_board yes)
-    (property "Reference" "#PWR092" (id 0) (at 101.6 121.92 0)
+    (property "Reference" "#PWR079" (id 0) (at 101.6 121.92 0)
       (effects (font (size 1.27 1.27)) hide)
     )
@@
       (effects (font (size 1.27 1.27)) hide)
     )
+    (pin "1")
   )
-  (symbol (lib_id "Device:R") (at 93.98 107.95 0)
+  (symbol (lib_id "Device:R") (at 93.98 107.95 0) (unit 1)
     (in_bom yes) (on_board yes)
-    (property "Reference" "R39" (id 0) (at 95.7581 106.8006 0)
+    (property "Reference" "R33" (id 0) (at 95.7581 106.8006 0)
       (effects (font (size 1.27 1.27)) (justify left))
     )
@@
       (effects (font (size 1.27 1.27)) hide)
     )
+    (pin "1")
+    (pin "2")
   )
-  (symbol (lib_id "Device:R") (at 101.6 88.9 0)
+  (symbol (lib_id "TCY_IC:UT6MA2TCR") (at 109.22 92.71 0) (unit 2)
     (in_bom yes) (on_board yes)
-    (property "Reference" "R40" (id 0) (at 103.3781 87.7506 0)
+    (property "Reference" "Q4" (id 0) (at 113.1571 85.2106 0)
+      (effects (font (size 1.27 1.27)) (justify left))
+    )
+    (property "Value" "UT6MA2TCR" (id 1) (at 115.6971 97.6693 90)
+      (effects (font (size 1.27 1.27)) (justify left))
+    )
+    (property "Footprint" "TCY_IC:UDFN-6-2EP_2x2mm_P0.65mm_EP1x0.7mm" (id 2) (at 113.03 107.95 0)
+      (effects (font (size 1.27 1.27) italic) hide)
+    )
+    (property "Datasheet" "https://cz.mouser.com/datasheet/2/348/ut6ma2tcr-e-1873584.pdf" (id 3) (at 114.3 110.49 0)
+      (effects (font (size 1.27 1.27)) hide)
+    )
+    (pin "1")
+    (pin "2")
+    (pin "6")
+    (pin "7")
+    (pin "3")
+    (pin "4")
+    (pin "5")
+    (pin "8")
+  )
+  (symbol (lib_id "TCY_IC:UT6MA2TCR") (at 99.06 100.33 0) (unit 1)
+    (in_bom yes) (on_board yes)
+    (property "Reference" "Q4" (id 0) (at 95.3771 94.1006 0)
+      (effects (font (size 1.27 1.27)) (justify left))
+    )
+    (property "Value" "UT6MA2TCR" (id 1) (at 89.0271 96.3993 0)
+      (effects (font (size 1.27 1.27)) (justify left))
+    )
+    (property "Footprint" "TCY_IC:UDFN-6-2EP_2x2mm_P0.65mm_EP1x0.7mm" (id 2) (at 102.87 115.57 0)
+      (effects (font (size 1.27 1.27) italic) hide)
+    )
+    (property "Datasheet" "https://cz.mouser.com/datasheet/2/348/ut6ma2tcr-e-1873584.pdf" (id 3) (at 104.14 118.11 0)
+      (effects (font (size 1.27 1.27)) hide)
+    )
+    (pin "1")
+    (pin "2")
+    (pin "6")
+    (pin "7")
+    (pin "3")
+    (pin "4")
+    (pin "5")
+    (pin "8")
+  )
+  (symbol (lib_id "Device:R") (at 101.6 88.9 0) (unit 1)
+    (in_bom yes) (on_board yes)
+    (property "Reference" "R34" (id 0) (at 103.3781 87.7506 0)
       (effects (font (size 1.27 1.27)) (justify left))
     )
@@
       (effects (font (size 1.27 1.27)) hide)
     )
-  )
-  (symbol (lib_id "TCY_IC:UT6MA2TCR") (at 99.06 100.33 0)
-    (in_bom yes) (on_board yes)
-    (property "Reference" "Q6" (id 0) (at 95.3771 94.1006 0)
-      (effects (font (size 1.27 1.27)) (justify left))
-    )
-    (property "Value" "UT6MA2TCR" (id 1) (at 89.0271 96.3993 0)
-      (effects (font (size 1.27 1.27)) (justify left))
-    )
-    (property "Footprint" "TCY_IC:UDFN-6-2EP_2x2mm_P0.65mm_EP1x0.7mm" (id 2) (at 102.87 115.57 0)
-      (effects (font (size 1.27 1.27) italic) hide)
-    )
-    (property "Datasheet" "https://cz.mouser.com/datasheet/2/348/ut6ma2tcr-e-1873584.pdf" (id 3) (at 104.14 118.11 0)
-      (effects (font (size 1.27 1.27)) hide)
-    )
-  )
-  (symbol (lib_id "TCY_IC:UT6MA2TCR") (at 109.22 92.71 0)
-    (in_bom yes) (on_board yes)
-    (property "Reference" "Q6" (id 0) (at 113.1571 85.2106 0)
-      (effects (font (size 1.27 1.27)) (justify left))
-    )
-    (property "Value" "UT6MA2TCR" (id 1) (at 115.6971 97.6693 90)
-      (effects (font (size 1.27 1.27)) (justify left))
-    )
-    (property "Footprint" "TCY_IC:UDFN-6-2EP_2x2mm_P0.65mm_EP1x0.7mm" (id 2) (at 113.03 107.95 0)
-      (effects (font (size 1.27 1.27) italic) hide)
-    )
-    (property "Datasheet" "https://cz.mouser.com/datasheet/2/348/ut6ma2tcr-e-1873584.pdf" (id 3) (at 114.3 110.49 0)
-      (effects (font (size 1.27 1.27)) hide)
-    )
+    (pin "1")
+    (pin "2")
   )
 )
